File: i2c_proto_petal_workshop/sao_proto.kicad_pcb (KiCad board)
At the start: 2 copper layers, 41 x 55.4 mm, 32 parts, among them J1 Simple_Addon_v2, J2 Programming: Jump Me, J3 GPIOs, J4 Jumpers, U1 CH32V003FxPx

Commit message: updated schematic
Parts:
- moved J3 2.55 mm to (151.8, 120.0), turned to 90 degrees

Commit message: added Mitch's schematic revision, layout images and 3D step file for the potentiometer
Parts:
- added D2: METRO LED, LED_THT:LED_D5.0mm, B.Cu at (103.1, 84.8)
- added D3: 1N4001, Diode_THT:D_DO-41_SOD81_P10.16mm_Horizontal, B.Cu at (81.9, 108.5)
- added M1: Vibro Motor PWM, Connector_PinHeader_1.00mm:PinHeader_1x02_P1.00mm_Vertical, B.Cu at (101.9, 111.8)
- added Q1: 2N2222 (NPN), Package_TO_SOT_THT:TO-92_Inline_Wide, B.Cu at (99.6, 103.9)
- added R2: 220R, Resistor_THT:R_Axial_DIN0309_L9.0mm_D3.2mm_P12.70mm_Horizontal, B.Cu at (81.6, 94.5)
- added R3: 10K, Resistor_THT:R_Axial_DIN0309_L9.0mm_D3.2mm_P12.70mm_Horizontal, B.Cu at (81.6, 99.2)
- added R4: 1K, Resistor_THT:R_Axial_DIN0309_L9.0mm_D3.2mm_P12.70mm_Horizontal, B.Cu at (81.6, 104.0)
- added RV1: 10K, Potentiometer_THT:Potentiometer_Alps_RK09Y11_Single_Horizontal, B.Cu at (96.2, 84.1)
- added SW1: SW_Push, Button_Switch_THT:SW_PUSH_6mm, B.Cu at (98.7, 97.3)
- D1: value LED -> REC LED
- J2, J3: footprint Library:PinHeader_1x02_P2.54mm -> Connector_PinHeader_2.54mm:PinHeader_1x02_P2.54mm_Vertical
- J4: footprint Library:PinHeader_1x14_P2.54mm -> Connector_PinHeader_2.54mm:PinHeader_1x14_P2.54mm_Vertical
- R1: renamed from R2; value R -> 1K
Connections:
- net Net-(J1-SCL) renamed /PC2
- net Net-(J1-SDA) renamed /PC1
- net Net-(J2-Pin_1) renamed /PD1
- net Net-(U1-PD0) renamed /PD0
- J1 pad 6: Net-(J1-GPIO2) -> /PC0
- J3 pad 1: Net-(J1-GPIO2) -> Net-(J1-GPIO1)
- J3 pad 2: Net-(J1-GPIO1) -> /PC0
Routing:
- net Net-(J1-GPIO2): track 9.92 -> 0.00 mm
- net /PC0: track 29.5 -> 39.4 mm
